Commit message: add hardware_type

File: urdf/crane_x7.ros2_control.xacro (robot description, xacro)
@@ -32,8 +32,16 @@
             manipulator_config_file_path
             manipulator_links_file_path
+	    initial_positions_file
+	    hardware_type
             ">
+    <xacro:property name="initial_positions" value="${xacro.load_yaml(initial_positions_file)['initial_positions']}"/>
     <ros2_control name="${name}" type="system">
       <hardware>
-        <plugin>crane_x7_hardware/CraneX7Hardware</plugin>
+	<xacro:if value="${hardware_type == 'mock'}">
+	  <plugin>mock_components/GenericSystem</plugin>
+  	</xacro:if>
+	<xacro:if value="${hardware_type == 'real'}">
+	  <plugin>crane_x7_hardware/CraneX7Hardware</plugin>
+  	</xacro:if>
         <param name="port_name">${port_name}</param>
         <param name="baudrate">${baudrate}</param>
@@ -47,5 +55,7 @@
           <param name="max">${joint_1_upper_limit}</param>
         </command_interface>
-        <state_interface name="position"/>
+        <state_interface name="position">
+          <param name="initial_value">${initial_positions['crane_x7_shoulder_fixed_part_pan_joint']}</param>
+	</state_interface>
         <state_interface name="velocity"/>
         <state_interface name="effort"/>
@@ -57,5 +67,7 @@
           <param name="max">${joint_2_upper_limit}</param>
         </command_interface>
-        <state_interface name="position"/>
+        <state_interface name="position">
+          <param name="initial_value">${initial_positions['crane_x7_shoulder_revolute_part_tilt_joint']}</param>
+	</state_interface>
         <state_interface name="velocity"/>
         <state_interface name="effort"/>
@@ -67,5 +79,7 @@
           <param name="max">${joint_3_upper_limit}</param>
         </command_interface>
-        <state_interface name="position"/>
+        <state_interface name="position">
+          <param name="initial_value">${initial_positions['crane_x7_upper_arm_revolute_part_twist_joint']}</param>
+	</state_interface>
         <state_interface name="velocity"/>
         <state_interface name="effort"/>
@@ -77,5 +91,7 @@
           <param name="max">${joint_4_upper_limit}</param>
         </command_interface>
-        <state_interface name="position"/>
+        <state_interface name="position">
+          <param name="initial_value">${initial_positions['crane_x7_upper_arm_revolute_part_rotate_joint']}</param>
+	</state_interface>
         <state_interface name="velocity"/>
         <state_interface name="effort"/>
@@ -87,5 +103,7 @@
           <param name="max">${joint_5_upper_limit}</param>
         </command_interface>
-        <state_interface name="position"/>
+        <state_interface name="position">
+          <param name="initial_value">${initial_positions['crane_x7_lower_arm_fixed_part_joint']}</param>
+	</state_interface>
         <state_interface name="velocity"/>
         <state_interface name="effort"/>
@@ -97,5 +115,7 @@
           <param name="max">${joint_6_upper_limit}</param>
         </command_interface>
-        <state_interface name="position"/>
+        <state_interface name="position">
+          <param name="initial_value">${initial_positions['crane_x7_lower_arm_revolute_part_joint']}</param>
+	</state_interface>
         <state_interface name="velocity"/>
         <state_interface name="effort"/>
@@ -107,5 +127,7 @@
           <param name="max">${joint_7_upper_limit}</param>
         </command_interface>
-        <state_interface name="position"/>
+        <state_interface name="position">
+          <param name="initial_value">${initial_positions['crane_x7_wrist_joint']}</param>
+	</state_interface>
         <state_interface name="velocity"/>
         <state_interface name="effort"/>

File: urdf/crane_x7.urdf.xacro (robot description, xacro)
@@ -20,4 +20,6 @@
   <xacro:arg name="gz_control_config_package" default="" />
   <xacro:arg name="gz_control_config_file_path" default="" />
+  <xacro:arg name="initial_positions_file" default="$(find crane_x7_description)/urdf/initial_positions.yaml"/>
+  <xacro:arg name="hardware_type" default="mock" />
   <!-- Link to provide the location reference for the arm -->
   <link name="base_link"/>
@@ -205,4 +207,6 @@
       manipulator_config_file_path="$(arg manipulator_config_file_path)"
       manipulator_links_file_path="$(arg manipulator_links_file_path)"
+      initial_positions_file="$(arg initial_positions_file)"
+      hardware_type="$(arg hardware_type)"
       />
   </xacro:unless>
